Commit message: remove localization

File: race_station_description/urdf/base.urdf (robot description, URDF)
Before this commit: robot race_station, 10 links, 9 joints
Joints:
- joint apriltag0_joint: origin xyz=1.2 0.4 0.0 rpy=0.0 0.0 0.0 -> xyz=1.1 0.4 0.0 rpy=0.0 0.0 1.5707963
- joint apriltag1_joint: origin xyz=0.15 0.4 0.0 rpy=0.0 0.0 0.0 -> xyz=0.2 0.4 0.0 rpy=0.0 0.0 1.5707963
- joint apriltag2_joint: origin xyz=1.4 0.4 -0.3 rpy=0.0 1.5707963 0.0 -> xyz=0.0 0.4 0.3 rpy=1.5707963 0.0 1.5707963

Commit message: dock point

File: race_station_description/urdf/base.urdf (robot description, URDF)
Before this commit: robot race_station, 10 links, 9 joints
Links:
- added link dockpoint
Joints:
- added joint dockpoint_joint: type fixed, parent base_link, child dockpoint, origin xyz=0.6 0.4 0.0 rpy=0.0 0.0 0.0
