Commit message: update

File: race_station_description/urdf/base.urdf (robot description, URDF)
Before this commit: robot race_station, 11 links, 10 joints
Links:
- removed link apriltag0
- removed link apriltag1
- removed link apriltag2
- added link apriltag25h9_02
- added link apriltag25h9_13
- added link apriltag25h9_17
- added link apriltag25h9_25
- added link apriltag36h11_009
- added link apriltag36h11_022
- added link apriltag36h11_2
- added link apriltag36h11_3
- added link apriltag36h11_4
- added link apriltag36h11_5
- added link apriltag36h11_6
- added link apriltag36h11_7
- added link apriltag36h11_8
- added link apriltag36h11_9
Joints:
- removed joint apriltag0_joint
- removed joint apriltag1_joint
- removed joint apriltag2_joint
- added joint apriltag25h9_02_joint: type fixed, parent base_link, child apriltag25h9_02, origin xyz=0.0 0.33 0.17 rpy=0.0 1.5707963 0.0
- added joint apriltag25h9_13_joint: type fixed, parent base_link, child apriltag25h9_13, origin xyz=-0.65 0.68 0.17 rpy=1.5707963 1.5707963 3.1415926
- added joint apriltag25h9_17_joint: type fixed, parent base_link, child apriltag25h9_17, origin xyz=-1.22 0.33 0.17 rpy=0.0 1.5707963 3.1415926
- added joint apriltag25h9_25_joint: type fixed, parent base_link, child apriltag25h9_25, origin xyz=-0.65 -0.03 0.17 rpy=1.5707963 1.5707963 0.0
- added joint apriltag36h11_009_joint: type fixed, parent base_link, child apriltag36h11_009, origin xyz=-0.42 0.12 0.0 rpy=0.0 3.1415926 3.1415926
- added joint apriltag36h11_022_joint: type fixed, parent base_link, child apriltag36h11_022, origin xyz=-0.42 0.52 0.0 rpy=0.0 3.1415926 3.1415926
- added joint apriltag36h11_2_joint: type fixed, parent base_link, child apriltag36h11_2, origin xyz=0.0 0.0 0.0 rpy=0.0 0.0 0.0
- added joint apriltag36h11_3_joint: type fixed, parent base_link, child apriltag36h11_3, origin xyz=0.0 0.0 0.0 rpy=0.0 0.0 0.0
- added joint apriltag36h11_4_joint: type fixed, parent base_link, child apriltag36h11_4, origin xyz=0.0 0.0 0.0 rpy=0.0 0.0 0.0
- added joint apriltag36h11_5_joint: type fixed, parent base_link, child apriltag36h11_5, origin xyz=0.0 0.0 0.0 rpy=0.0 0.0 0.0
- added joint apriltag36h11_6_joint: type fixed, parent base_link, child apriltag36h11_6, origin xyz=0.0 0.0 0.0 rpy=0.0 0.0 0.0
- added joint apriltag36h11_7_joint: type fixed, parent base_link, child apriltag36h11_7, origin xyz=0.0 0.0 0.0 rpy=0.0 0.0 0.0
- added joint apriltag36h11_8_joint: type fixed, parent base_link, child apriltag36h11_8, origin xyz=0.0 0.0 0.0 rpy=0.0 0.0 0.0
- added joint apriltag36h11_9_joint: type fixed, parent base_link, child apriltag36h11_9, origin xyz=0.0 0.0 0.0 rpy=0.0 0.0 0.0

Commit message: update dock point tf

File: race_station_description/urdf/base.urdf (robot description, URDF)
Before this commit: robot race_station, 22 links, 21 joints
Links:
- removed link apriltag36h11_2
- removed link apriltag36h11_3
- removed link apriltag36h11_4
- removed link apriltag36h11_5
- removed link apriltag36h11_6
- removed link apriltag36h11_7
- removed link apriltag36h11_8
- removed link apriltag36h11_9
- removed link dockpoint
- added link dock_point
Joints:
- removed joint apriltag36h11_2_joint
- removed joint apriltag36h11_3_joint
- removed joint apriltag36h11_4_joint
- removed joint apriltag36h11_5_joint
- removed joint apriltag36h11_6_joint
- removed joint apriltag36h11_7_joint
- removed joint apriltag36h11_8_joint
- removed joint apriltag36h11_9_joint
- removed joint dockpoint_joint
- added joint dock_point_joint: type fixed, parent base_link, child dock_point, origin xyz=-0.415 0.33 -0.05 rpy=0.0 0.0 0.0

Commit message: updated sim

File: race_station_description/urdf/base.urdf (robot description, URDF)
Before this commit: robot race_station, 14 links, 13 joints
Links:
- removed link apriltag25h9_25
- removed link apriltag36h11_009
- removed link apriltag36h11_022
- added link apriltag36h11_146
- added link apriltag36h11_176
- added link apriltag36h11_185
- added link apriltag36h11_541
- added link apriltag36h11_558
Joints:
- removed joint apriltag25h9_25_joint
- removed joint apriltag36h11_009_joint
- removed joint apriltag36h11_022_joint
- added joint apriltag36h11_146_joint: type fixed, parent dock_point, child apriltag36h11_146, origin xyz=0.430 0.0 0.405 rpy=0.0 1.5707963 0.0
- added joint apriltag36h11_176_joint: type fixed, parent dock_point, child apriltag36h11_176, origin xyz=0.0 0.25 -0.012 rpy=0.0 0.0 0.0
- added joint apriltag36h11_185_joint: type fixed, parent dock_point, child apriltag36h11_185, origin xyz=0.0 -0.25 -0.012 rpy=0.0 0.0 0.0
- added joint apriltag36h11_541_joint: type fixed, parent dock_point, child apriltag36h11_541, origin xyz=0.470 0.0 0.160 rpy=0.0 1.5707963 0.0
- added joint apriltag36h11_558_joint: type fixed, parent dock_point, child apriltag36h11_558, origin xyz=0.470 0.0 0.095 rpy=0.0 1.5707963 0.0
- joint apriltag25h9_02_joint: origin xyz=0.0 0.33 0.17 rpy=0.0 1.5707963 0.0 -> xyz=-0.81 0.0 -0.21 rpy=0.0 1.5707963 0.0; parent base_link -> dock_point
- joint apriltag25h9_13_joint: origin xyz=-0.65 0.68 0.17 rpy=1.5707963 1.5707963 3.1415926 -> xyz=-0.26 0.37 -0.21 rpy=1.5707963 1.5707963 0.0; parent base_link -> dock_point
- joint apriltag25h9_17_joint: origin xyz=-1.22 0.33 0.17 rpy=0.0 1.5707963 3.1415926 -> xyz=-0.26 -0.37 -0.21 rpy=-1.5707963 1.5707963 0.0; parent base_link -> dock_point
- joint dock_point_joint: origin xyz=-0.415 0.33 -0.05 rpy=0.0 0.0 0.0 -> xyz=-0.410 0.325 -0.04 rpy=3.1415926 0.0 0.0

Commit message: updated apriltags tf

File: race_station_description/urdf/base.urdf (robot description, URDF)
Before this commit: robot race_station, 16 links, 15 joints
Joints:
- joint apriltag25h9_02_joint: origin xyz=-0.81 0.0 -0.21 rpy=0.0 1.5707963 0.0 -> xyz=-0.81 0.0 -0.21 rpy=-1.5707963 0.0 -1.5707963
- joint apriltag25h9_13_joint: origin xyz=-0.26 0.37 -0.21 rpy=1.5707963 1.5707963 0.0 -> xyz=-0.26 0.37 -0.21 rpy=-1.5707963 0.0 3.1415926
- joint apriltag25h9_17_joint: origin xyz=-0.26 -0.37 -0.21 rpy=-1.5707963 1.5707963 0.0 -> xyz=-0.26 -0.37 -0.21 rpy=-1.5707963 0.0 0.0
- joint apriltag36h11_146_joint: origin xyz=0.430 0.0 0.405 rpy=0.0 1.5707963 0.0 -> xyz=0.430 0.0 0.405 rpy=-1.5707963 0.0 -1.5707963
- joint apriltag36h11_176_joint: origin xyz=0.0 0.25 -0.012 rpy=0.0 0.0 0.0 -> xyz=0.0 0.25 -0.012 rpy=3.1415926 0.0 -1.5707963
- joint apriltag36h11_185_joint: origin xyz=0.0 -0.25 -0.012 rpy=0.0 0.0 0.0 -> xyz=0.0 -0.25 -0.012 rpy=3.1415926 0.0 -1.5707963
- joint apriltag36h11_541_joint: origin xyz=0.470 0.0 0.160 rpy=0.0 1.5707963 0.0 -> xyz=0.470 0.0 0.160 rpy=-1.5707963 0.0 -1.5707963
- joint apriltag36h11_558_joint: origin xyz=0.470 0.0 0.095 rpy=0.0 1.5707963 0.0 -> xyz=0.470 0.0 0.095 rpy=-1.5707963 0.0 -1.5707963
